File: projects/arduino/arduino.brd (EAGLE design)
At the start: 205.7 x 131.8 mm, 33 parts

Commit message: update
Parts:
- removed MCP1: MCP2515, MCP2515:MCP2515
- added MCP2: MCP2515, MCP2515:MCP2515
- moved LED2 88.8 mm to (-24.1, -16.5)
- moved R6 80.7 mm to (-16.5, -16.5)
- moved C2 72.0 mm to (0.00, -16.5)
- moved C1 71.8 mm to (0.00, -19.1)
- moved C4 68.7 mm to (5.08, -16.5)
- moved C3 68.4 mm to (5.08, -19.1)
- moved R5 66.3 mm to (-43.2, -15.2)
- moved IM1 60.3 mm to (-39.4, 1.27)
- moved U$3 57.4 mm to (12.7, -19.1)
- moved R1 55.1 mm to (17.8, -5.08)
- moved R2 55.1 mm to (17.8, -7.62)
- moved R3 55.1 mm to (17.8, -10.2)
- moved R4 55.1 mm to (17.8, -12.7)
- moved LED1 52.2 mm to (-34.3, -16.5)
- moved IM2 45.6 mm to (-10.2, 1.27)
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Connections:
- net +5V: now also MCP2.VDD; no longer MCP1.VDD
- net CAN_INT: now also MCP2.INT; no longer MCP1.INT
- net MISO: now also MCP2.SO; no longer MCP1.SO
- net MOSI: now also MCP2.SI; no longer MCP1.SI
- net N$1: now also MCP2.OSC2; no longer MCP1.OSC2
- net N$2: now also MCP2.OSC1; no longer MCP1.OSC1
- net N$3: now also MCP2.TXCAN; no longer MCP1.TXCAN
- net N$4: now also MCP2.RXCAN; no longer MCP1.RXCAN
- net N$5: now also MCP2.RESET; no longer MCP1.RESET
- net SCLK: now also MCP2.SCK; no longer MCP1.SCK
- net SS: now also MCP2.CS; no longer MCP1.CS
- net V-: now also MCP2.VSS; no longer MCP1.VSS
Routing:
- net V-: track 445.9 -> 0.00 mm, vias 2 -> 0
- net +5V: track 396.4 -> 0.00 mm
- net GND: track 136.1 -> 0.00 mm, vias 1 -> 0
- net IM_RESET: track 130.8 -> 0.00 mm, vias 1 -> 0
- net PWM4: track 122.9 -> 0.00 mm
- net DIR2: track 118.5 -> 0.00 mm
- net IM_BUSY: track 104.0 -> 0.00 mm, vias 1 -> 0
- net STBY: track 91.0 -> 0.00 mm
- net IM_BUSY2: track 68.6 -> 0.00 mm, vias 1 -> 0
- net PWM3: track 63.9 -> 0.00 mm
- net N$11: track 59.4 -> 0.00 mm
- net DIR1: track 58.2 -> 0.00 mm, vias 1 -> 0
- net IM_RESET2: track 50.0 -> 0.00 mm, vias 1 -> 0
- net N$2: track 42.7 -> 0.00 mm
- net PWM2: track 41.7 -> 0.00 mm
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Other:
- board size 205.7 x 131.8 mm -> 147.3 x 122 mm
