File: projects/arduino/arduino.sch (EAGLE design)
At the start: 33 parts

Commit message: update
Parts:
- renumbered MCP1 to MCP2
Changed lines of the file:
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@@
 <parts>
 <part name="B1" library="ArduinoMega" deviceset="ARDUINO_ARDUINO_MEGA_R3" device="FULL" override_package3d_urn="urn:adsk.eagle:package:38784594/2" override_package_urn="urn:adsk.eagle:footprint:38784595/1"/>
-<part name="U$1" library="MCP2562" deviceset="MCP2562" device="" override_package3d_urn="urn:adsk.eagle:package:38785330/2" override_package_urn="urn:adsk.eagle:footprint:38785331/1"/>
-<part name="MCP1" library="MCP2515" deviceset="MCP2515" device="" override_package3d_urn="urn:adsk.eagle:package:38784723/2" override_package_urn="urn:adsk.eagle:footprint:38784724/1"/>
+<part name="U$1" library="MCP2562" deviceset="MCP2562" device="" override_package3d_urn="urn:adsk.eagle:package:38785330/2" override_package_urn="urn:adsk.eagle:footprint:38785331/1" override_locally_modified="yes"/>
 <part name="U$2" library="Module" deviceset="MD13S" device="" override_package3d_urn="urn:adsk.eagle:package:38784770/2" override_package_urn="urn:adsk.eagle:footprint:38784774/1"/>
 <part name="U$3" library="HUSG20" deviceset="HUSG20" device="" override_package3d_urn="urn:adsk.eagle:package:38791805/2" override_package_urn="urn:adsk.eagle:footprint:38791806/1"/>
@@
 <part name="P+1" library="supply1" library_urn="urn:adsk.eagle:library:371" deviceset="+5V" device=""/>
 <part name="IM1" library="IM920" deviceset="IM920C" device="" override_package3d_urn="urn:adsk.eagle:package:38786354/2" override_package_urn="urn:adsk.eagle:footprint:38786355/1"/>
-<part name="IM2" library="IM920" deviceset="IM920" device="IM920_BOARD" override_package3d_urn="urn:adsk.eagle:package:38786734/2" override_package_urn="urn:adsk.eagle:footprint:38786772/1"/>
+<part name="IM2" library="IM920" deviceset="IM920" device="IM920_BOARD" override_package3d_urn="urn:adsk.eagle:package:38786734/2" override_package_urn="urn:adsk.eagle:footprint:38786772/1" override_locally_modified="yes"/>
 <part name="P+2" library="supply1" library_urn="urn:adsk.eagle:library:371" deviceset="+5V" device=""/>
 <part name="R1" library="rcl" library_urn="urn:adsk.eagle:library:334" deviceset="R-EU_" device="0207/10" package3d_urn="urn:adsk.eagle:package:23491/2"/>
@@
 <part name="R6" library="rcl" library_urn="urn:adsk.eagle:library:334" deviceset="R-EU_" device="0207/10" package3d_urn="urn:adsk.eagle:package:23491/2"/>
 <part name="GND3" library="supply1" library_urn="urn:adsk.eagle:library:371" deviceset="GND" device=""/>
+<part name="MCP2" library="MCP2515" deviceset="MCP2515" device=""/>
 </parts>
 <sheets>
@@
 </instance>
 <instance part="U$1" gate="G$1" x="195.58" y="71.12" smashed="yes"/>
-<instance part="MCP1" gate="G$1" x="200.66" y="111.76" smashed="yes"/>
 <instance part="U$2" gate="G$1" x="15.24" y="68.58" smashed="yes">
 <attribute name="MPN" x="5.08" y="76.962" size="1.778" layer="96"/>
@@
 <attribute name="VALUE" x="297.18" y="-20.32" size="1.778" layer="96" rot="R90"/>
 </instance>
+<instance part="MCP2" gate="G$1" x="200.66" y="111.76" smashed="yes"/>
 </instances>
 <busses>
@@
 <net name="N$1" class="0">
 <segment>
-<pinref part="MCP1" gate="G$1" pin="OSC2"/>
 <pinref part="U$3" gate="G$1" pin="A"/>
 <wire x1="187.96" y1="99.06" x2="165.1" y2="99.06" width="0.1524" layer="91"/>
@@
 <pinref part="C1" gate="G$1" pin="1"/>
 <wire x1="154.94" y1="99.06" x2="154.94" y2="96.52" width="0.1524" layer="91"/>
+<pinref part="MCP2" gate="G$1" pin="OSC2"/>
 </segment>
 </net>
 <net name="N$2" class="0">
 <segment>
-<pinref part="MCP1" gate="G$1" pin="OSC1"/>
 <wire x1="187.96" y1="96.52" x2="177.8" y2="96.52" width="0.1524" layer="91"/>
 <wire x1="177.8" y1="96.52" x2="177.8" y2="81.28" width="0.1524" layer="91"/>
@@
 <junction x="165.1" y="81.28"/>
 <wire x1="165.1" y1="78.74" x2="154.94" y2="78.74" width="0.1524" layer="91"/>
+<pinref part="MCP2" gate="G$1" pin="OSC1"/>
 </segment>
 </net>
@@
 <pinref part="U$1" gate="G$1" pin="TXD"/>
 <wire x1="187.96" y1="81.28" x2="180.34" y2="81.28" width="0.1524" layer="91"/>
-<pinref part="MCP1" gate="G$1" pin="TXCAN"/>
 <wire x1="180.34" y1="81.28" x2="180.34" y2="114.3" width="0.1524" layer="91"/>
 <wire x1="180.34" y1="114.3" x2="187.96" y2="114.3" width="0.1524" layer="91"/>
+<pinref part="MCP2" gate="G$1" pin="TXCAN"/>
 </segment>
 </net>
 <net name="N$4" class="0">
 <segment>
-<pinref part="MCP1" gate="G$1" pin="RXCAN"/>
 <wire x1="187.96" y1="111.76" x2="182.88" y2="111.76" width="0.1524" layer="91"/>
 <pinref part="U$1" gate="G$1" pin="RXD"/>
 <wire x1="182.88" y1="111.76" x2="182.88" y2="73.66" width="0.1524" layer="91"/>
 <wire x1="182.88" y1="73.66" x2="187.96" y2="73.66" width="0.1524" layer="91"/>
+<pinref part="MCP2" gate="G$1" pin="RXCAN"/>
 </segment>
 </net>
@@
 </segment>
 <segment>
-<pinref part="MCP1" gate="G$1" pin="VSS"/>
 <pinref part="P-2" gate="1" pin="GND"/>
 <wire x1="187.96" y1="93.98" x2="185.42" y2="93.98" width="0.1524" layer="91"/>
 <wire x1="185.42" y1="93.98" x2="185.42" y2="88.9" width="0.1524" layer="91"/>
+<pinref part="MCP2" gate="G$1" pin="VSS"/>
 </segment>
 <segment>
@@
 </segment>
 <segment>
-<pinref part="MCP1" gate="G$1" pin="VDD"/>
 <pinref part="R1" gate="G$1" pin="2"/>
 <wire x1="243.84" y1="111.76" x2="243.84" y2="114.3" width="0.1524" layer="91"/>
@@
 <wire x1="223.52" y1="127" x2="223.52" y2="114.3" width="0.1524" layer="91"/>
 <junction x="223.52" y="114.3"/>
+<pinref part="MCP2" gate="G$1" pin="VDD"/>
 </segment>
 </net>
 <net name="SS" class="0">
 <segment>
-<pinref part="MCP1" gate="G$1" pin="CS"/>
 <wire x1="218.44" y1="106.68" x2="226.06" y2="106.68" width="0.1524" layer="91"/>
 <label x="226.06" y="106.68" size="1.778" layer="95" xref="yes"/>
+<pinref part="MCP2" gate="G$1" pin="CS"/>
 </segment>
 <segment>
@@
 <net name="MOSI" class="0">
 <segment>
-<pinref part="MCP1" gate="G$1" pin="SI"/>
 <wire x1="218.44" y1="104.14" x2="226.06" y2="104.14" width="0.1524" layer="91"/>
 <label x="226.06" y="104.14" size="1.778" layer="95" xref="yes"/>
+<pinref part="MCP2" gate="G$1" pin="SI"/>
 </segment>
 <segment>
@@
 <net name="SCLK" class="0">
 <segment>
-<pinref part="MCP1" gate="G$1" pin="SCK"/>
 <wire x1="218.44" y1="101.6" x2="226.06" y2="101.6" width="0.1524" layer="91"/>
 <label x="226.06" y="101.6" size="1.778" layer="95" xref="yes"/>
+<pinref part="MCP2" gate="G$1" pin="SCK"/>
 </segment>
 <segment>
@@
 <net name="MISO" class="0">
 <segment>
-<pinref part="MCP1" gate="G$1" pin="SO"/>
 <wire x1="218.44" y1="109.22" x2="226.06" y2="109.22" width="0.1524" layer="91"/>
 <label x="226.06" y="109.22" size="1.778" layer="95" xref="yes"/>
+<pinref part="MCP2" gate="G$1" pin="SO"/>
 </segment>
 <segment>
@@
 <net name="N$5" class="0">
 <segment>
-<pinref part="MCP1" gate="G$1" pin="RESET"/>
 <pinref part="R1" gate="G$1" pin="1"/>
 <wire x1="218.44" y1="111.76" x2="233.68" y2="111.76" width="0.1524" layer="91"/>
+<pinref part="MCP2" gate="G$1" pin="RESET"/>
 </segment>
 </net>
@@
 <net name="CAN_INT" class="0">
 <segment>
-<pinref part="MCP1" gate="G$1" pin="INT"/>
 <wire x1="218.44" y1="99.06" x2="226.06" y2="99.06" width="0.1524" layer="91"/>
 <label x="226.06" y="99.06" size="1.778" layer="95" xref="yes"/>
-</segment>
-</net>
+<pinref part="MCP2" gate="G$1" pin="INT"/>
+</segment>
+</net>

Commit message: changeArduino
Parts:
- removed C4: (no value), rcl:C-EU025-024X044
- removed POW, POW1, POW2, POW3, POW4: (no value), XR Connector:2PIN_SIDE
- removed R4: (no value), rcl:R-EU_0207/10
- removed S2: (no value), switch-dil:DS01E
- added CAN1, CAN2, CAN3, MOTOR_LF, MOTOR_LR, MOTOR_RF, MOTOR_RR: (no value), TB113-2B-x-x-0-x-x:2PIN
- renumbered U$2 to DRIVER_RF, U$4 to DRIBER_RR, U$5 to DRIVER_LF, U$6 to DRIVER_LR
Connections:
- removed net N$12: POW4.P$1, R4.2
- removed net N$9: S2.1, U$1.CANL
- net +5V: now also MOTOR_LF.P$2, MOTOR_LR.P$2, MOTOR_RF.P$2, MOTOR_RR.P$2; no longer POW.P$1, POW1.P$1, POW2.P$1, POW3.P$1
- net GND: now also R2.2
- net N$11: now also CAN1.P$2, CAN2.P$2, CAN3.P$2, U$1.CANL; no longer C4.1, R2.2, R4.1, S1.2, S2.2
- net N$7: now also CAN1.P$1, CAN2.P$1, CAN3.P$1, S1.2, U$1.CANH; no longer POW4.P$2, R3.2
- net N$8: now also R3.2; no longer U$1.CANH
- net V-: now also MOTOR_LF.P$1, MOTOR_LR.P$1, MOTOR_RF.P$1, MOTOR_RR.P$1; no longer C4.2, POW.P$2, POW1.P$2, POW2.P$2, POW3.P$2
Other:
- moved on the sheet: R3, S1
