File: projects/jetson/Jetson Nano.brd (EAGLE design)
At the start: 102.8 x 82.2 mm, 19 parts, among them X1 MKDSN1,5/4-5,08, X2 MKDSN1,5/4-5,08

Commit message: change all
Parts:
- removed C4: (no value), rcl:C025-024X044
- removed R4: (no value), rcl:0207/10
- removed S1, S2: (no value), switch-dil:DS-01
- removed X1, X2: MKDSN1,5/4-5,08, con-phoenix-508:MKDSN1,5/4-5,08
- added 5VIN1, 5VIN2, CAN1, CAN2: (no value), TB113-2B-x-x-0-x-x:2PIN
- added R5, R6: (no value), rcl:0207/10
- added SW: SRIDE_SWITCH, Sride Switch:SRIDE_SWITCH
- moved R3 25.7 mm to (82.5, 2.54)
Connections:
- removed net 3.3V: C3.1, JN1.3V3-1, MCP1.VDD, R1.2, U$1.VCC, U$2.1_VIN, U$3.3.3V, U$4.VDD
- removed net 5V_1: JN1.5V-1, U$3.5V, X1.1
- removed net CAN_H: R3.2, X1.3, X2.3
- removed net CAN_H3: C4.1, R2.2, R3.1, R4.1, S1.2, S2.2
- removed net CAN_L: R4.2, X1.4, X2.4
- new net +3V3: JN1.3V3-1, MCP1.VDD, R1.2, R5.2, R6.2, U$1.VCC, U$2.1_VIN, U$3.3.3V
- new net +5V: 5VIN1.P$1, C3.1, JN1.5V-1, U$3.5V, U$4.VDD
- new net N$1: R2.2
- new net N$15: R3.2, SW.R
- net 5V_2: now also 5VIN2.P$1; no longer X2.1
- net CAN_H2: now also CAN1.P$1, CAN2.P$1, SW.LR; no longer S1.1
- net CAN_INT: now also R5.1
- net N$16: now also CAN1.P$2, CAN2.P$2, R3.1; no longer S2.1
- net N$2: now also 5VIN1.P$2, 5VIN2.P$2; no longer U$3.GND, X1.2, X2.2
- net SS: now also R6.1
- net V-: no longer C4.2
Routing:
- net 3.3V: track 151.1 -> 0.00 mm
- net CAN_L: track 133.2 -> 0.00 mm
- net N$2: track 128.6 -> 0.00 mm
- net CAN_H: track 109.9 -> 0.00 mm
- net 5V_1: track 108.9 -> 0.00 mm
- net CAN_H3: track 69.1 -> 0.00 mm
- net V-: track 68.8 -> 0.00 mm
- net N$4: track 63.5 -> 0.00 mm
- net N$3: track 53.3 -> 0.00 mm
- net N$7: track 40.5 -> 0.00 mm
- net N$12: track 40.3 -> 0.00 mm
- net N$11: track 40.3 -> 0.00 mm
- net N$14: track 38.4 -> 0.00 mm
- net N$5: track 29.0 -> 0.00 mm
- net 5V_2: track 23.7 -> 0.00 mm
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Other:
- board size 102.8 x 82.2 mm -> 97.8 x 82.2 mm

Commit message: add
Parts:
- moved CAN2 137.9 mm to (20.3, 77.5)
- moved U$3 76.4 mm to (78.7, 68.6)
- moved R3 67.4 mm to (36.8, 52.1), turned to 90 degrees
- moved R1 65.4 mm to (21.6, 52.1), turned to 90 degrees
- moved CAN1 62.5 mm to (61.0, 3.81), turned to 180 degrees
- moved 5VIN2 59.7 mm to (43.2, 3.81), turned to 180 degrees
- moved R2 56.9 mm to (29.2, 52.1), turned to 90 degrees
- moved R6 51.0 mm to (52.1, 52.1), turned to 90 degrees
- moved R5 49.5 mm to (44.5, 52.1), turned to 90 degrees
- moved U$4 25.4 mm to (80.0, 26.7), turned to 180 degrees
- moved 5VIN1 22.6 mm to (24.1, 3.81), turned to 180 degrees
- moved C3 20.7 mm to (58.4, 52.1), turned to 270 degrees
- moved C2 15.9 mm to (64.8, 52.1), turned to 270 degrees
- moved U$1 15.3 mm to (38.1, 39.4), turned to 270 degrees
- moved C1 13.7 mm to (71.1, 52.1), turned to 270 degrees
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Routing:
- net +5V: track 0.00 -> 187.5 mm, vias 0 -> 1
- net CAN_H2: track 0.00 -> 179.2 mm, vias 0 -> 2
- net +3V3: track 0.00 -> 141.3 mm
- net N$16: track 0.00 -> 125.8 mm
- net N$15: track 0.00 -> 94.9 mm
- net N$2: track 0.00 -> 88.9 mm
- net V-: track 0.00 -> 77.4 mm
- net N$12: track 0.00 -> 74.2 mm
- net N$11: track 0.00 -> 74.2 mm
- net N$7: track 0.00 -> 70.7 mm
- net 5V_2: track 0.00 -> 65.6 mm
- net N$14: track 0.00 -> 55.5 mm
- net N$5: track 0.00 -> 52.1 mm
- net N$13: track 0.00 -> 49.5 mm
- net N$4: track 0.00 -> 46.8 mm
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Other:
- board size 97.8 x 82.2 mm -> 118.1 x 93.6 mm

Commit message: jet
Parts:
- moved U$3 4.58 mm to (74.9, 66.0)
Routing:
- net +5V: track 187.5 -> 205.9 mm
- net N$12: track 74.2 -> 71.4 mm
- net +3V3: track 141.3 -> 138.9 mm
- net N$11: track 74.2 -> 71.8 mm
Other:
- board size 118.1 x 93.6 mm -> 120 x 100 mm
