File: projects/power_supply/power.brd (EAGLE design)
At the start: 135.9 x 98.7 mm, 91 parts, among them SW1 SRIDE_SWITCH, SW2 SRIDE_SWITCH, SW3 SRIDE_SWITCH, SW4 SRIDE_SWITCH, SW5 SRIDE_SWITCH, SW6 SRIDE_SWITCH, SW7 SRIDE_SWITCH, SW8 SRIDE_SWITCH

Commit message: NISHIMOTO_TAKENORI
Parts:
- removed L2: (no value), Chip LED:OSXX1608C1A
- removed R12, R16, R23, R25, R28, R32, R4, R8: 100k, rcl:R0603
- removed U$12, U$15, U$18, U$19, U$22, U$26, U$6, U$9: 2SJ334, 2SJ334:2SJ334
- added ARDUINO-OUT1, ARDUINO-OUT2, ARDUINO-OUT3, JETSON-OUT1: (no value), TB113-2B-x-x-0-x-x:2PIN
- added MM: (no value), Chip LED:OSXX1608C1A
- moved EMERGENCY 116.4 mm to (8.89, -3.81), turned to 180 degrees
- moved BIO-OUT 87.5 mm to (35.6, -3.81), turned to 180 degrees
- moved MOTOR-FL-OUT 85.0 mm to (135.9, -3.81), turned to 180 degrees
- moved ARM-OUT 74.0 mm to (61.0, -3.81), turned to 180 degrees
- moved JETSON-OUT 73.3 mm to (193.0, 76.2)
- moved MOTOR-RR-OUT 70.6 mm to (111.8, -3.81), turned to 180 degrees
- moved MOTOR-RL-OUT 66.2 mm to (86.4, -3.81), turned to 180 degrees
- moved BIO-IN 54.6 mm to (160.0, 90.2)
- moved U$25 53.5 mm to (154.9, 66.0)
- moved U$24 53.3 mm to (154.9, 77.5)
- moved ARDUINO-IN 45.4 mm to (67.0, 90.0)
- moved ARM-IN 41.9 mm to (133.3, 90.2)
- moved U$21 40.7 mm to (128.3, 64.8)
- moved U$20 40.7 mm to (128.3, 76.2)
- moved R1 39.5 mm to (120.7, 11.4)
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Connections:
- net N$11 renamed MS
- net N$12 renamed MU
- net N$17 renamed MJUY
- net N$2 renamed MKK
- net N$20 renamed MH
- net N$21 renamed MY
- net N$22 renamed MV
- net N$26 renamed MDSDS
- net N$29 renamed MBV
- net N$3 renamed MBB
- net N$30 renamed MX
- net N$31 renamed MHH
- net N$35 renamed MHHHH
- net N$38 renamed MCX
- net N$39 renamed MN
- net N$4 renamed MOO
- net N$40 renamed MZZ
- net N$44 renamed MA
- net N$45 renamed 18V
- net N$47 renamed MAC
- net N$53 renamed MVVV
- net N$54 renamed MGG
- net N$55 renamed MHGF
- removed net GND: EMERGENCY.P$1
- removed net N$16: MOTOR-FR-OUT.P$2, R6.2, R8.1, SW2.LR, U$7.GATE, U$9.SOURCE
- removed net N$25: MOTOR-FL-OUT.P$2, R10.2, R12.1, SW3.LR, U$10.GATE, U$12.SOURCE
- removed net N$27: MOTOR-FL-IN.P$1, U$12.DRAIN
- removed net N$34: MOTOR-RR-OUT.P$2, R14.2, R16.1, SW4.LR, U$13.GATE, U$15.SOURCE
- removed net N$36: MOTOR-RR-IN.P$1, U$15.DRAIN
- removed net N$46: MOTOR-RL-OUT.P$2, R18.2, R23.1, SW5.LR, U$16.GATE, U$18.SOURCE
- removed net N$51: MOTOR-RL-IN.P$1, U$18.DRAIN
- removed net N$57: JETSON-OUT.P$2, R20.2, R25.1, SW6.LR, U$19.SOURCE, U$3.GATE
- removed net N$59: JETSON-IN.P$1, U$19.DRAIN
- removed net N$61: ARM-OUT.P$2, R26.2, R28.1, SW7.LR, U$20.GATE, U$22.SOURCE
- removed net N$63: ARM-IN.P$1, U$22.DRAIN
- removed net N$64: BIO-OUT.P$2, R30.2, R32.1, SW8.LR, U$24.GATE, U$26.SOURCE
- removed net N$65: EMERGENCY.P$2, R12.2, R16.2, R23.2, R25.2, R28.2, R32.2, R4.2, R8.2, U$12.GATE, U$15.GATE, U$18.GATE, U$19.GATE, U$22.GATE, U$26.GATE, U$6.GATE, U$9.GATE
- removed net N$66: BIO-IN.P$1, U$26.DRAIN
- removed net N$7: ARDUINO-OUT.P$2, R2.2, R4.1, SW1.LR, U$1.GATE, U$6.SOURCE
- new net IN: ARDUINO-IN.P$1, ARDUINO-OUT.P$2, ARM-IN.P$1, ARM-OUT.P$2, BIO-IN.P$1, BIO-OUT.P$2, EMERGENCY.P$1, JETSON-IN.P$1, JETSON-OUT.P$2, MOTOR-FL-IN.P$1, MOTOR-FL-OUT.P$2, MOTOR-FR-IN.P$1, MOTOR-FR-OUT.P$2, MOTOR-RL-IN.P$1, MOTOR-RL-OUT.P$2, MOTOR-RR-IN.P$1, MOTOR-RR-OUT.P$2, R10.2, R14.2, R18.2, R2.2, R20.2, R26.2, R30.2, R6.2, U$1.GATE, U$10.GATE, U$13.GATE, U$16.GATE, U$20.GATE, U$24.GATE, U$3.GATE, U$7.GATE
- new net MAD: JETSON-OUT1.P$1
- new net ML: ARDUINO-OUT1.P$1, ARDUINO-OUT2.P$1, ARDUINO-OUT3.P$1
- new net OUT: EMERGENCY.P$2, SW1.LR, SW2.LR, SW3.LR, SW4.LR, SW5.LR, SW6.LR, SW7.LR, SW8.LR
- net N$13: now also MM.AN; no longer L2.AN
- net N$14: now also MM.CT; no longer L2.CT
- net N$18: now also JETSON-OUT1.P$2; no longer MOTOR-FR-IN.P$1, U$9.DRAIN
- net N$9: now also ARDUINO-OUT1.P$2, ARDUINO-OUT2.P$2, ARDUINO-OUT3.P$2; no longer ARDUINO-IN.P$1, U$6.DRAIN
Routing:
- net N$65: track 256.3 -> 0.00 mm, vias 5 -> 0
- net N$57: track 203.7 -> 0.00 mm, vias 1 -> 0
- net N$25: track 182.5 -> 0.00 mm, vias 1 -> 0
- net N$34: track 168.2 -> 0.00 mm, vias 1 -> 0
- net MV: track 166.6 -> 0.00 mm, vias 2 -> 0
- net MOO: track 159.4 -> 0.00 mm
- net MAC: track 148.4 -> 0.00 mm, vias 4 -> 0
- net N$7: track 143.2 -> 0.00 mm
- net MKK: track 141.4 -> 0.00 mm, vias 1 -> 0
- net N$16: track 141.3 -> 0.00 mm, vias 1 -> 0
- net N$46: track 141.0 -> 0.00 mm, vias 1 -> 0
- net N$64: track 139.1 -> 0.00 mm, vias 3 -> 0
- net MA: track 129.0 -> 0.00 mm, vias 1 -> 0
- net MHH: track 122.8 -> 0.00 mm
- net N$61: track 106.2 -> 0.00 mm, vias 4 -> 0
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Other:
- board size 135.9 x 98.7 mm -> 208.3 x 115.2 mm

Commit message: ka
Parts:
- removed ARDUINO-OUT, ARDUINO-OUT1, ARDUINO-OUT2, ARDUINO-OUT3, JETSON-OUT, JETSON-OUT1: (no value), TB113-2B-x-x-0-x-x:2PIN
- added ARDUINO18V-OUT, ARDUINO5V-IN, ARDUINO5V-OUT1, ARDUINO5V-OUT2, ARDUINO5V-OUT3, JETSON18V-OUT, JETSON5V-IN, JETSON5V-OUT1, JETSON5V-OUT2: (no value), TB113-2B-x-x-0-x-x:2PIN
- moved U$23 124.3 mm to (61.0, 151.1)
- moved MOTOR-FR-OUT 120.7 mm to (160.0, -3.00), turned to 180 degrees
- moved U$2 99.7 mm to (-19.1, 139.7)
- moved BIO-IN 30.0 mm to (190.0, 90.0)
- moved EMERGENCY 28.9 mm to (-20.0, -3.00)
- moved JETSON-IN 27.0 mm to (-20.0, 90.0)
- moved ARM-IN 26.7 mm to (160.0, 90.0)
- moved BIO-OUT 25.6 mm to (10.0, -3.00)
- moved ARM-OUT 21.0 mm to (40.0, -3.00)
- moved MOTOR-RL-IN 19.5 mm to (130.0, 90.0)
- moved MOTOR-FR-IN 18.1 mm to (10.0, 90.0)
- moved MOTOR-RL-OUT 16.4 mm to (70.0, -3.00)
- moved MOTOR-RR-IN 12.4 mm to (100.0, 90.0)
- moved MOTOR-RR-OUT 11.8 mm to (100.0, -3.00)
- moved MOTOR-FL-IN 8.26 mm to (40.0, 90.0)
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Connections:
- net IN: now also ARDUINO18V-OUT.P$2, JETSON18V-OUT.P$2; no longer ARDUINO-OUT.P$2, JETSON-OUT.P$2
- net MAC: now also JETSON18V-OUT.P$1; no longer JETSON-OUT.P$1
- net MAD: now also JETSON5V-IN.P$1, JETSON5V-OUT1.P$1, JETSON5V-OUT2.P$1; no longer JETSON-OUT1.P$1
- net ML: now also ARDUINO5V-IN.P$1, ARDUINO5V-OUT1.P$1, ARDUINO5V-OUT2.P$1, ARDUINO5V-OUT3.P$1; no longer ARDUINO-OUT1.P$1, ARDUINO-OUT2.P$1, ARDUINO-OUT3.P$1
- net MOO: now also ARDUINO18V-OUT.P$1; no longer ARDUINO-OUT.P$1
- net N$18: now also JETSON5V-IN.P$2, JETSON5V-OUT1.P$2, JETSON5V-OUT2.P$2; no longer JETSON-OUT1.P$2
- net N$9: now also ARDUINO5V-IN.P$2, ARDUINO5V-OUT1.P$2, ARDUINO5V-OUT2.P$2, ARDUINO5V-OUT3.P$2; no longer ARDUINO-OUT1.P$2, ARDUINO-OUT2.P$2, ARDUINO-OUT3.P$2
Routing:
- net N$1: track 98.0 -> 0.00 mm
- net N$8: track 89.4 -> 0.00 mm
- net N$52: track 67.8 -> 0.00 mm
- net N$10: track 66.2 -> 0.00 mm
- net N$9: track 62.7 -> 0.00 mm
- net N$43: track 62.3 -> 0.00 mm
- net N$19: track 52.0 -> 0.00 mm
- net N$28: track 50.2 -> 0.00 mm
- net N$37: track 48.7 -> 0.00 mm
Other:
- board size 208.3 x 115.2 mm -> 298.4 x 115.2 mm

Commit message: power
Parts:
- removed L1, L3, L4, L5, L6, L7, L8, MM: (no value), Chip LED:OSXX1608C1A
- removed R26, R27, R29, R30, R31: 100k, rcl:R0603
- added LED2, LED3, LED4, LED5, LED6, LED7, LED8, LED9: (no value), led:LED5MM
- added R12, R16, R23, R4, R8: (no value), resistor-power:AC01
- R1, R10, R11, R13, R14, R15, R17, R18, R19, R2, R20, R21, R22, R24, R3, R5, R6, R7, R9: value 100k -> (none); device rcl:R0603 -> resistor-power:AC01
- moved EMERGENCY 285.8 mm to (265.8, -1.73)
- moved ARDUINO18V-OUT 205.5 mm to (-10.2, 22.9)
- moved BIO-OUT 180.3 mm to (190.3, -3.00)
- moved SW8 175.1 mm to (250.2, 91.4)
- moved SW7 174.1 mm to (250.2, 80.0)
- moved SW6 173.3 mm to (250.2, 67.3)
- moved SW5 172.8 mm to (250.2, 55.9)
- moved SW4 172.2 mm to (250.2, 43.2)
- moved SW3 171.8 mm to (250.2, 31.8)
- moved SW2 171.5 mm to (250.2, 19.1)
- moved SW1 171.5 mm to (250.2, 6.35)
- moved U$23 150.9 mm to (-33.0, 33.0)
- moved JETSON18V-OUT 139.3 mm to (-10.2, 44.5)
- moved ARM-OUT 119.4 mm to (159.4, -3.00)
- moved MOTOR-FR-OUT 118.1 mm to (41.9, -3.00)
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Connections:
- removed net N$14: MM.CT, R7.2
- removed net N$23: L3.CT, R11.2
- removed net N$32: L4.CT, R15.2
- removed net N$41: L5.CT, R22.2
- removed net N$48: L7.CT, R21.2
- removed net N$5: L1.CT, R3.2
- removed net N$50: L8.CT, R31.2
- removed net N$56: L6.CT, R27.2
- removed net N$60 (its old number): R26.1, R27.1
- new net N$11: LED6.A, R15.2
- new net N$12: LED7.A, R18.2
- new net N$16: LED8.A, R21.2
- new net N$17: LED9.A, R24.2
- new net N$2: LED2.A, R2.2
- new net N$3: LED3.A, R6.2
- new net N$4: LED4.A, R9.2
- new net N$49: R1.1, R2.1
- new net N$7: LED5.A, R12.2
- net IN: now also LED2.K, LED3.K, LED4.K, LED5.K, LED6.K, LED7.K, LED8.K, LED9.K; no longer R10.2, R14.2, R18.2, R2.2, R20.2, R26.2, R30.2, R6.2
- net MA: now also R4.2; no longer R19.2
- net MAC: now also R1.2; no longer L7.AN
- net MCX: now also R16.2; no longer R17.2
- net MH: now also R10.2; no longer R9.2
- net MHGF: now also R20.2; no longer L6.AN
- net MHH: now also R14.2; no longer L4.AN
- net MHHHH: now also R23.2; no longer L8.AN
- net MJUY: now also R22.2; no longer R29.2
- net MKK: now also R3.2; no longer R1.2
- net MOO: now also R5.2; no longer L1.AN
- net MS: now also R7.2; no longer R5.2
- net MV: now also R11.2; no longer L3.AN
- net MVVV: now also R19.2; no longer R24.2
- net MZZ: now also R17.2; no longer L5.AN
- net N$1: now also R3.1; no longer R1.1
- net N$10: now also R7.1; no longer R5.1
- net N$13: now also R8.2; no longer MM.AN
- net N$15: now also R8.1, R9.1; no longer R6.1, R7.1
- net N$19: now also R10.1; no longer R9.1
- net N$24: now also R12.1; no longer R10.1
- net N$37: now also R16.1; no longer R17.1
- net N$42: now also R17.1; no longer R22.1
- net N$43: now also R4.1; no longer R19.1
- net N$52: now also R19.1; no longer R24.1
- net N$58: now also R23.1, R24.1; no longer R30.1, R31.1
- net N$6: now also R5.1, R6.1; no longer R2.1, R3.1
- net N$8: now also R22.1; no longer R29.1
Other:
- board size 298.4 x 115.2 mm -> 402.6 x 115.2 mm

Commit message: k
Parts:
- moved LED9 305.7 mm to (170.2, 11.4), turned to 90 degrees
- moved LED8 281.6 mm to (147.3, 11.4), turned to 90 degrees
- moved LED7 258.7 mm to (125.7, 11.4), turned to 90 degrees
- moved LED6 238.3 mm to (106.7, 11.4), turned to 90 degrees
- moved LED5 217.9 mm to (87.6, 11.4), turned to 90 degrees
- moved LED4 197.5 mm to (68.6, 11.4), turned to 90 degrees
- moved LED3 177.1 mm to (49.5, 11.4), turned to 90 degrees
- moved LED2 159.3 mm to (33.0, 11.4), turned to 90 degrees
- moved R1 5.08 mm to (29.2, 35.6)
- moved R10 5.08 mm to (90.2, 35.6)
- moved R11 5.08 mm to (97.8, 35.6)
- moved R12 5.08 mm to (105.4, 35.6)
- moved R13 5.08 mm to (113.0, 35.6)
- moved R14 5.08 mm to (120.7, 35.6)
- moved R15 5.08 mm to (128.3, 35.6)
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Routing:
- net IN: track 0.00 -> 783.2 mm
- net N$43: track 0.00 -> 363.6 mm
- net N$1: track 0.00 -> 263.9 mm, vias 0 -> 1
- net N$10: track 0.00 -> 234.3 mm, vias 0 -> 1
- net N$19: track 0.00 -> 204.7 mm
- net N$28: track 0.00 -> 178.1 mm, vias 0 -> 1
- net N$37: track 0.00 -> 156.7 mm, vias 0 -> 1
- net N$52: track 0.00 -> 134.5 mm, vias 0 -> 1
- net N$8: track 0.00 -> 113.3 mm, vias 0 -> 1
- net OUT: track 0.00 -> 106.0 mm
- net N$13: track 0.00 -> 105.3 mm, vias 0 -> 1
- net MV: track 0.00 -> 95.0 mm
- net N$12: track 0.00 -> 91.3 mm
- net MOO: track 0.00 -> 90.3 mm, vias 0 -> 1
- net MHH: track 0.00 -> 88.9 mm, vias 0 -> 1
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
Commit message: anya
Routing:
- net N$43: track 363.6 -> 314.3 mm, vias 0 -> 1
- net N$12: track 91.3 -> 51.3 mm
- net N$16: track 84.9 -> 52.8 mm
- net N$13: track 105.3 -> 129.2 mm, vias 1 -> 0
- net MDSDS: track 34.9 -> 18.5 mm
- net N$11: track 58.9 -> 44.3 mm
- net N$10: track 234.3 -> 246.0 mm, vias 1 -> 0
- net IN: track 783.2 -> 793.4 mm
- net N$7: track 50.4 -> 41.7 mm
- net ML: track 80.0 -> 71.6 mm
- net N$8: track 113.3 -> 121.3 mm, vias 1 -> 0
- net MZZ: track 81.0 -> 73.2 mm
- net MHH: track 88.9 -> 82.2 mm, vias 1 -> 0
- net N$4: track 46.5 -> 40.1 mm
- net N$28: track 178.1 -> 183.1 mm, vias 1 -> 0
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
Commit message: a
Parts:
- added JETSON5V-IN1: (no value), TB113-2B-x-x-0-x-x:2PIN
- added U$6: DCDCDEV, dcdcDEVkit:DCDCDEV
Connections:
- net MAD: now also JETSON5V-IN1.P$2
- net N$18: now also JETSON5V-IN1.P$1
Changed lines of the file:
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@@
 <attribute name="VALUE" x="171.9834" y="14.6304" size="1.27" layer="27" ratio="10" rot="R90"/>
+</element>
+<element name="U$6" library="dcdcDEVkit" package="DCDCDEV" package3d_urn="urn:adsk.eagle:package:38731238/2" value="DCDCDEV" x="-124.46" y="-38.1" smashed="yes"/>
+<element name="JETSON5V-IN1" library="TB113-2B-x-x-0-x-x" library_urn="urn:adsk.eagle:library:38507486" package="2PIN" package3d_urn="urn:adsk.eagle:package:38507490/6" override_package3d_urn="urn:adsk.eagle:package:38731294/2" override_package_urn="urn:adsk.eagle:footprint:38731295/1" value="" x="-119.38" y="-49.53" smashed="yes">
+<attribute name="NAME" x="-124.46" y="-41.91" size="1.27" layer="21"/>
 </element>
 </elements>
@@
 <wire x1="-112.9284" y1="87.5538" x2="-113.03" y2="87.63" width="2.54" layer="1"/>
 <wire x1="-112.4712" y1="63.3222" x2="-112.9284" y2="62.1792" width="2.54" layer="1"/>
+<contactref element="JETSON5V-IN1" pad="P$2"/>
+<wire x1="-88.9" y1="57.15" x2="-116.84" y2="-49.53" width="0" layer="19" extent="1-1"/>
 </signal>
 <signal name="N$18" class="1">
@@
 <wire x1="-112.9284" y1="92.583" x2="-113.03" y2="92.71" width="2.54" layer="16"/>
 <wire x1="-112.4712" y1="68.3514" x2="-113.03" y2="67.31" width="2.54" layer="16"/>
+<contactref element="JETSON5V-IN1" pad="P$1"/>
+<wire x1="-88.9" y1="52.07" x2="-121.92" y2="-49.53" width="0" layer="19" extent="1-1"/>
 </signal>
 <signal name="N$49">
