File: projects/power_supply/power.sch (EAGLE design)
At the start: 91 parts, among them SW1 SRIDE_SWITCH, SW2 SRIDE_SWITCH, SW3 SRIDE_SWITCH, SW4 SRIDE_SWITCH, SW5 SRIDE_SWITCH, SW6 SRIDE_SWITCH, SW7 SRIDE_SWITCH, SW8 SRIDE_SWITCH

Commit message: NISHIMOTO_TAKENORI
Parts:
- removed L2: (no value), Chip LED:OSXX1608C1A
- removed R12, R16, R23, R25, R28, R32, R4, R8: 100k, rcl:R-US_R0603
- removed U$12, U$15, U$18, U$19, U$22, U$26, U$6, U$9: 2SJ334, 2SJ334:2SJ334
- added ARDUINO-OUT1, ARDUINO-OUT2, ARDUINO-OUT3, JETSON-OUT1: (no value), TB113-2B-x-x-0-x-x:2PIN
- added MM: (no value), Chip LED:OSXX1608C1A
Connections:
- net N$11 renamed MS
- net N$12 renamed MU
- net N$17 renamed MJUY
- net N$2 renamed MKK
- net N$20 renamed MH
- net N$21 renamed MY
- net N$22 renamed MV
- net N$26 renamed MDSDS
- net N$29 renamed MBV
- net N$3 renamed MBB
- net N$30 renamed MX
- net N$31 renamed MHH
- net N$35 renamed MHHHH
- net N$38 renamed MCX
- net N$39 renamed MN
- net N$4 renamed MOO
- net N$40 renamed MZZ
- net N$44 renamed MA
- net N$45 renamed 18V
- net N$47 renamed MAC
- net N$53 renamed MVVV
- net N$54 renamed MGG
- net N$55 renamed MHGF
- removed net GND: EMERGENCY.P$1
- removed net N$16: MOTOR-FR-OUT.P$2, R6.2, R8.1, SW2.LR, U$7.GATE, U$9.SOURCE
- removed net N$25: MOTOR-FL-OUT.P$2, R10.2, R12.1, SW3.LR, U$10.GATE, U$12.SOURCE
- removed net N$27: MOTOR-FL-IN.P$1, U$12.DRAIN
- removed net N$34: MOTOR-RR-OUT.P$2, R14.2, R16.1, SW4.LR, U$13.GATE, U$15.SOURCE
- removed net N$36: MOTOR-RR-IN.P$1, U$15.DRAIN
- removed net N$46: MOTOR-RL-OUT.P$2, R18.2, R23.1, SW5.LR, U$16.GATE, U$18.SOURCE
- removed net N$51: MOTOR-RL-IN.P$1, U$18.DRAIN
- removed net N$57: JETSON-OUT.P$2, R20.2, R25.1, SW6.LR, U$19.SOURCE, U$3.GATE
- removed net N$59: JETSON-IN.P$1, U$19.DRAIN
- removed net N$61: ARM-OUT.P$2, R26.2, R28.1, SW7.LR, U$20.GATE, U$22.SOURCE
- removed net N$63: ARM-IN.P$1, U$22.DRAIN
- removed net N$64: BIO-OUT.P$2, R30.2, R32.1, SW8.LR, U$24.GATE, U$26.SOURCE
- removed net N$65: EMERGENCY.P$2, R12.2, R16.2, R23.2, R25.2, R28.2, R32.2, R4.2, R8.2, U$12.GATE, U$15.GATE, U$18.GATE, U$19.GATE, U$22.GATE, U$26.GATE, U$6.GATE, U$9.GATE
- removed net N$66: BIO-IN.P$1, U$26.DRAIN
- removed net N$7: ARDUINO-OUT.P$2, R2.2, R4.1, SW1.LR, U$1.GATE, U$6.SOURCE
- new net IN: ARDUINO-IN.P$1, ARDUINO-OUT.P$2, ARM-IN.P$1, ARM-OUT.P$2, BIO-IN.P$1, BIO-OUT.P$2, EMERGENCY.P$1, JETSON-IN.P$1, JETSON-OUT.P$2, MOTOR-FL-IN.P$1, MOTOR-FL-OUT.P$2, MOTOR-FR-IN.P$1, MOTOR-FR-OUT.P$2, MOTOR-RL-IN.P$1, MOTOR-RL-OUT.P$2, MOTOR-RR-IN.P$1, MOTOR-RR-OUT.P$2, R10.2, R14.2, R18.2, R2.2, R20.2, R26.2, R30.2, R6.2, U$1.GATE, U$10.GATE, U$13.GATE, U$16.GATE, U$20.GATE, U$24.GATE, U$3.GATE, U$7.GATE
- new net MAD: JETSON-OUT1.P$1
- new net ML: ARDUINO-OUT1.P$1, ARDUINO-OUT2.P$1, ARDUINO-OUT3.P$1
- new net OUT: EMERGENCY.P$2, SW1.LR, SW2.LR, SW3.LR, SW4.LR, SW5.LR, SW6.LR, SW7.LR, SW8.LR
- net N$13: now also MM.AN; no longer L2.AN
- net N$14: now also MM.CT; no longer L2.CT
- net N$18: now also JETSON-OUT1.P$2; no longer MOTOR-FR-IN.P$1, U$9.DRAIN
- net N$9: now also ARDUINO-OUT1.P$2, ARDUINO-OUT2.P$2, ARDUINO-OUT3.P$2; no longer ARDUINO-IN.P$1, U$6.DRAIN
Other:
- moved on the sheet: ARDUINO-IN, ARDUINO-OUT, ARM-IN, ARM-OUT, BIO-IN, BIO-OUT, JETSON-OUT, L1, L3, L4, L5, L6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

Commit message: ka
Parts:
- removed ARDUINO-OUT1, ARDUINO-OUT3: (no value), TB113-2B-x-x-0-x-x:2PIN
- added ARDUINO5V-OUT1, ARDUINO5V-OUT2, ARDUINO5V-OUT3, JETSON5V-OUT1, JETSON5V-OUT2: (no value), TB113-2B-x-x-0-x-x:2PIN
- renumbered ARDUINO-OUT to ARDUINO18V-OUT, ARDUINO-OUT2 to ARDUINO5V-IN, JETSON-OUT to JETSON18V-OUT, JETSON-OUT1 to JETSON5V-IN
Connections:
- net MAD: now also JETSON5V-OUT1.P$1, JETSON5V-OUT2.P$1
- net ML: now also ARDUINO5V-OUT1.P$1, ARDUINO5V-OUT2.P$1, ARDUINO5V-OUT3.P$1; no longer ARDUINO-OUT1.P$1, ARDUINO-OUT3.P$1
- net N$18: now also JETSON5V-OUT1.P$2, JETSON5V-OUT2.P$2
- net N$9: now also ARDUINO5V-OUT1.P$2, ARDUINO5V-OUT2.P$2, ARDUINO5V-OUT3.P$2; no longer ARDUINO-OUT1.P$2, ARDUINO-OUT3.P$2

Commit message: power
Parts:
- removed L1, L3, L4, L5, L6, L7, L8, MM: (no value), Chip LED:OSXX1608C1A
- removed R26, R27, R29, R30, R31: 100k, rcl:R-US_R0603
- added LED2, LED3, LED4, LED5, LED6, LED7, LED8, LED9: (no value), led:LED5MM
- added R12, R16, R23, R4, R8: (no value), resistor-power:RAC01
- R1, R10, R11, R13, R14, R15, R17, R18, R19, R2, R20, R21, R22, R24, R3, R5, R6, R7, R9: value 100k -> (none); device rcl:R-US_R0603 -> resistor-power:RAC01
Connections:
- removed net N$14: MM.CT, R7.2
- removed net N$23: L3.CT, R11.2
- removed net N$32: L4.CT, R15.2
- removed net N$41: L5.CT, R22.2
- removed net N$48: L7.CT, R21.2
- removed net N$5: L1.CT, R3.2
- removed net N$50: L8.CT, R31.2
- removed net N$56: L6.CT, R27.2
- removed net N$60 (its old number): R26.1, R27.1
- new net N$11: LED6.A, R15.2
- new net N$12: LED7.A, R18.2
- new net N$16: LED8.A, R21.2
- new net N$17: LED9.A, R24.2
- new net N$2: LED2.A, R2.2
- new net N$3: LED3.A, R6.2
- new net N$4: LED4.A, R9.2
- new net N$49: R1.1, R2.1
- new net N$7: LED5.A, R12.2
- net IN: now also LED2.C, LED3.C, LED4.C, LED5.C, LED6.C, LED7.C, LED8.C, LED9.C; no longer R10.2, R14.2, R18.2, R2.2, R20.2, R26.2, R30.2, R6.2
- net MA: now also R4.2; no longer R19.2
- net MAC: now also R1.2; no longer L7.AN
- net MCX: now also R16.2; no longer R17.2
- net MH: now also R10.2; no longer R9.2
- net MHGF: now also R20.2; no longer L6.AN
- net MHH: now also R14.2; no longer L4.AN
- net MHHHH: now also R23.2; no longer L8.AN
- net MJUY: now also R22.2; no longer R29.2
- net MKK: now also R3.2; no longer R1.2
- net MOO: now also R5.2; no longer L1.AN
- net MS: now also R7.2; no longer R5.2
- net MV: now also R11.2; no longer L3.AN
- net MVVV: now also R19.2; no longer R24.2
- net MZZ: now also R17.2; no longer L5.AN
- net N$1: now also R3.1; no longer R1.1
- net N$10: now also R7.1; no longer R5.1
- net N$13: now also R8.2; no longer MM.AN
- net N$15: now also R8.1, R9.1; no longer R6.1, R7.1
- net N$19: now also R10.1; no longer R9.1
- net N$24: now also R12.1; no longer R10.1
- net N$37: now also R16.1; no longer R17.1
- net N$42: now also R17.1; no longer R22.1
- net N$43: now also R4.1; no longer R19.1
- net N$52: now also R19.1; no longer R24.1
- net N$58: now also R23.1, R24.1; no longer R30.1, R31.1
- net N$6: now also R5.1, R6.1; no longer R2.1, R3.1
- net N$8: now also R22.1; no longer R29.1

Commit message: a
Parts:
- added JETSON5V-IN1: (no value), TB113-2B-x-x-0-x-x:2PIN
- added U$6: DCDCDEV, dcdcDEVkit:DCDCDEV
Connections:
- net MAD: now also JETSON5V-IN1.P$2
- net N$18: now also JETSON5V-IN1.P$1
Changed lines of the file:
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@@
 <part name="LED8" library="led" library_urn="urn:adsk.eagle:library:259" deviceset="LED" device="5MM" package3d_urn="urn:adsk.eagle:package:15799/2"/>
 <part name="LED9" library="led" library_urn="urn:adsk.eagle:library:259" deviceset="LED" device="5MM" package3d_urn="urn:adsk.eagle:package:15799/2"/>
+<part name="U$6" library="dcdcDEVkit" deviceset="DCDCDEV" device="" package3d_urn="urn:adsk.eagle:package:38731238/2"/>
+<part name="JETSON5V-IN1" library="TB113-2B-x-x-0-x-x" library_urn="urn:adsk.eagle:library:38507486" deviceset="2PIN" device="" package3d_urn="urn:adsk.eagle:package:38507490/6" override_package3d_urn="urn:adsk.eagle:package:38731294/2" override_package_urn="urn:adsk.eagle:footprint:38731295/1"/>
 </parts>
 <sheets>
@@
 <attribute name="NAME" x="115.316" y="-230.632" size="1.778" layer="95" rot="R90"/>
 <attribute name="VALUE" x="117.475" y="-230.632" size="1.778" layer="96" rot="R90"/>
+</instance>
+<instance part="U$6" gate="G$1" x="139.7" y="40.64" smashed="yes"/>
+<instance part="JETSON5V-IN1" gate="G$1" x="172.72" y="50.8" smashed="yes">
+<attribute name="NAME" x="170.18" y="55.88" size="1.27" layer="95"/>
 </instance>
 </instances>
@@
 <pinref part="JETSON5V-IN" gate="G$1" pin="P$1"/>
 <wire x1="172.72" y1="63.5" x2="172.72" y2="66.04" width="0.1524" layer="91"/>
-<wire x1="165.1" y1="63.5" x2="172.72" y2="63.5" width="0.1524" layer="91"/>
 <pinref part="JETSON5V-OUT1" gate="G$1" pin="P$1"/>
-<wire x1="172.72" y1="63.5" x2="190.5" y2="63.5" width="0.1524" layer="91"/>
+<wire x1="172.72" y1="63.5" x2="182.88" y2="63.5" width="0.1524" layer="91"/>
+<wire x1="182.88" y1="63.5" x2="190.5" y2="63.5" width="0.1524" layer="91"/>
 <wire x1="190.5" y1="63.5" x2="190.5" y2="66.04" width="0.1524" layer="91"/>
-<junction x="172.72" y="63.5"/>
 <wire x1="190.5" y1="63.5" x2="205.74" y2="63.5" width="0.1524" layer="91"/>
 <junction x="190.5" y="63.5"/>
 <pinref part="JETSON5V-OUT2" gate="G$1" pin="P$1"/>
 <wire x1="205.74" y1="63.5" x2="205.74" y2="66.04" width="0.1524" layer="91"/>
+<pinref part="JETSON5V-IN1" gate="G$1" pin="P$2"/>
+<wire x1="175.26" y1="45.72" x2="182.88" y2="45.72" width="0.1524" layer="91"/>
+<wire x1="182.88" y1="45.72" x2="182.88" y2="63.5" width="0.1524" layer="91"/>
+<junction x="182.88" y="63.5"/>
 </segment>
 </net>
@@
 <pinref part="JETSON5V-IN" gate="G$1" pin="P$2"/>
 <wire x1="175.26" y1="58.42" x2="175.26" y2="66.04" width="0.1524" layer="91"/>
-<wire x1="165.1" y1="58.42" x2="175.26" y2="58.42" width="0.1524" layer="91"/>
-<wire x1="175.26" y1="58.42" x2="193.04" y2="58.42" width="0.1524" layer="91"/>
-<junction x="175.26" y="58.42"/>
+<wire x1="175.26" y1="58.42" x2="187.96" y2="58.42" width="0.1524" layer="91"/>
 <pinref part="JETSON5V-OUT1" gate="G$1" pin="P$2"/>
+<wire x1="187.96" y1="58.42" x2="193.04" y2="58.42" width="0.1524" layer="91"/>
 <wire x1="193.04" y1="58.42" x2="193.04" y2="66.04" width="0.1524" layer="91"/>
 <wire x1="193.04" y1="58.42" x2="208.28" y2="58.42" width="0.1524" layer="91"/>
@@
 <pinref part="JETSON5V-OUT2" gate="G$1" pin="P$2"/>
 <wire x1="208.28" y1="58.42" x2="208.28" y2="66.04" width="0.1524" layer="91"/>
-</segment>
-</net>
+<pinref part="JETSON5V-IN1" gate="G$1" pin="P$1"/>
+<wire x1="172.72" y1="45.72" x2="172.72" y2="40.64" width="0.1524" layer="91"/>
+<wire x1="172.72" y1="40.64" x2="187.96" y2="40.64" width="0.1524" layer="91"/>
+<wire x1="187.96" y1="40.64" x2="187.96" y2="58.42" width="0.1524" layer="91"/>
+<junction x="187.96" y="58.42"/>
+</segment>
+</net>
