File: projects/power_supply/power_ver2.brd (EAGLE design)
At the start: 160 x 100 mm, 48 parts, among them SW1 SRIDE_SWITCH, SW6 SRIDE_SWITCH

Commit message: wakuwaku
Parts:
- removed ARDUINO5V-OUT3, ARM-IN, ARM-OUT, BIO-IN, BIO-OUT, JETSON5V-OUT2, MOTOR-FL-IN, MOTOR-FL-OUT, MOTOR-FR-IN, MOTOR-FR-OUT, MOTOR-RL-IN, MOTOR-RL-OUT, MOTOR-RR-IN, MOTOR-RR-OUT: (no value), TB113-2B-x-x-0-x-x:2PIN
- removed D1, D2, D3, D4, D5, D6, D7, D8: 1N5908, diode:C4111-15
- removed LED2, LED3: (no value), led:LED5MM
- removed SW1, SW6: SRIDE_SWITCH, Sride Switch:SRIDE_SWITCH
- added ARD, JET: SRIDE_SWITCH, Sride Switch:SRIDE_SWITCH
- added ARDUINO, JETSON: 1N5908, diode:C4111-15
- added A_ON, J_ON: (no value), led:LED5MM
- added JETSON18V-OUT1: (no value), TB113-2B-x-x-0-x-x:2PIN
- moved R6 197.9 mm to (97.0, 39.0), flipped to the bottom, turned to 90 degrees
- moved U$6 190.9 mm to (102.5, 20.4), turned to 90 degrees
- moved ARDUINO5V-OUT2 189.7 mm to (106.0, 69.0)
- moved R5 169.7 mm to (86.0, 39.0), flipped to the bottom, turned to 90 degrees
- moved ARDUINO5V-IN 144.3 mm to (91.0, 73.0), turned to 180 degrees
- moved ARDUINO5V-OUT1 143.2 mm to (76.0, 69.0)
- moved R2 137.6 mm to (33.0, 39.0), flipped to the bottom, turned to 90 degrees
- moved R4 136.4 mm to (67.0, 39.0), flipped to the bottom, turned to 90 degrees
- moved ARDUINO18V-OUT 126.3 mm to (91.9, 7.15)
- moved U$2 122.3 mm to (71.5, 20.5), turned to 90 degrees
- moved U$5 114.4 mm to (3.00, 63.0)
- moved JETSON18V-OUT 113.6 mm to (28.3, 7.15)
- moved R3 111.9 mm to (55.0, 39.0), flipped to the bottom, turned to 90 degrees
- moved R1 111.7 mm to (23.0, 39.0), flipped to the bottom, turned to 90 degrees
- moved JETSON5V-IN 110.6 mm to (61.0, 73.0), turned to 180 degrees
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Connections:
- removed net N$10: D2.C, MOTOR-FL-OUT.P$1
- removed net N$12: D3.A, MOTOR-RR-IN.P$2
- removed net N$13: D3.C, MOTOR-RR-OUT.P$1
- removed net N$15: D4.A, MOTOR-RL-IN.P$2
- removed net N$16: D4.C, MOTOR-RL-OUT.P$1
- removed net N$18: JETSON5V-IN.P$2, JETSON5V-IN1.P$1, JETSON5V-OUT1.P$2, JETSON5V-OUT2.P$2
- removed net N$19: ARM-IN.P$2, D5.A
- removed net N$20: ARM-OUT.P$1, D5.C
- removed net N$22: BIO-IN.P$2, D6.A
- removed net N$23: BIO-OUT.P$1, D6.C
- removed net N$4: D1.A, MOTOR-FR-IN.P$1
- removed net N$5: D1.C, MOTOR-FR-OUT.P$1
- removed net N$8: D2.A, MOTOR-FL-IN.P$2
- removed net N$9: ARDUINO5V-IN.P$2, ARDUINO5V-OUT1.P$2, ARDUINO5V-OUT2.P$2, ARDUINO5V-OUT3.P$2
- net 18V: now also JETSON.A; no longer D7.A
- net GND: now also ARDUINO5V-IN.P$2, ARDUINO5V-OUT1.P$2, ARDUINO5V-OUT2.P$2, A_ON.K, JETSON18V-OUT1.P$2, JETSON5V-IN.P$2, JETSON5V-IN1.P$2, JETSON5V-OUT1.P$2, J_ON.K; no longer ARM-IN.P$1, ARM-OUT.P$2, BIO-IN.P$1, BIO-OUT.P$2, LED2.K, LED3.K, MOTOR-FL-IN.P$1, MOTOR-FL-OUT.P$2, MOTOR-FR-IN.P$2, MOTOR-FR-OUT.P$2, MOTOR-RL-IN.P$1, MOTOR-RL-OUT.P$2, MOTOR-RR-IN.P$1, MOTOR-RR-OUT.P$2
- net MA: now also JETSON.C; no longer D7.C
- net MAC: now also JETSON18V-OUT1.P$1
- net MAD: now also JETSON5V-IN1.P$1; no longer JETSON5V-IN1.P$2, JETSON5V-OUT2.P$1
- net MBB: now also ARDUINO.A; no longer D8.A
- net MKK: now also ARDUINO.C; no longer D8.C
- net ML: no longer ARDUINO5V-OUT3.P$1
- net N$1: now also ARD.L; no longer SW1.L
- net N$2: now also J_ON.A; no longer LED2.A
- net N$3: now also A_ON.A; no longer LED3.A
- net N$43: now also JET.L; no longer SW6.L
- net OUT: now also ARD.LR, JET.LR; no longer SW1.LR, SW6.LR
Routing:
- net GND: track 0.00 -> 307.1 mm
- net N$43: track 0.00 -> 191.0 mm, vias 0 -> 1
- net OUT: track 0.00 -> 167.7 mm
- net N$1: track 0.00 -> 152.5 mm
- net MOO: track 0.00 -> 143.7 mm
- net MAC: track 0.00 -> 111.2 mm
- net MA: track 0.00 -> 101.4 mm
- net N$2: track 0.00 -> 89.7 mm
- net MKK: track 0.00 -> 86.2 mm, vias 0 -> 1
- net N$3: track 0.00 -> 38.4 mm
- net MAD: track 0.00 -> 38.3 mm
- net MBB: track 0.00 -> 35.9 mm
- net ML: track 0.00 -> 35.5 mm
- net 18V: track 0.00 -> 26.8 mm
- net N$6: track 0.00 -> 11.0 mm
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- added copper zone on layer 1, net GND
- added copper zone on layer 16, net GND
Other:
- board size 160 x 100 mm -> 140 x 80 mm

Commit message: aa
Parts:
- added JETSON1: 1N5908, diode:C4111-15
- added R7: (no value), resistor-power:AC01
- added U$1: 2SJ334, 2SJ334:2SJ334
- moved ARD 128.2 mm to (-10.0, 37.0), turned to 90 degrees
- moved JET 128.0 mm to (-10.0, 55.0), turned to 90 degrees
- moved A_ON 123.5 mm to (-5.00, 28.0), turned to 90 degrees
- moved J_ON 123.0 mm to (-5.00, 46.0), turned to 90 degrees
- moved ARDUINO 71.6 mm to (56.0, 72.0)
- moved ARDUINO5V-OUT2 47.9 mm to (63.0, 90.0)
- moved ARDUINO5V-OUT1 36.6 mm to (46.0, 90.0)
- moved JETSON 32.2 mm to (28.0, 72.0)
- moved ARDUINO-IN 30.0 mm to (-5.70, 68.0)
- moved JETSON5V-OUT1 29.7 mm to (24.0, 90.0)
- moved JETSON-IN 26.0 mm to (-5.60, 83.0)
- moved ARDUINO18V-OUT 22.2 mm to (69.9, 10.2)
- moved R5 21.1 mm to (65.0, 41.0)
- moved R6 21.1 mm to (76.0, 41.0)
- moved U$6 21.1 mm to (81.5, 22.4)
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Connections:
- removed net N$43: JET.L, R4.1, U$4.GATE
- new net MA1: JETSON1.C, R7.2, U$1.SOURCE
- new net N$4: JET.L, R4.1, R7.1, U$1.GATE, U$4.GATE
- new net N$5: JETSON18V-OUT1.P$1, U$1.DRAIN
- net 18V: now also JETSON1.A
- net MAC: no longer JETSON18V-OUT1.P$1
Routing:
- net GND: track 307.1 -> 0.00 mm
- net N$43: track 191.0 -> 0.00 mm, vias 1 -> 0
- net OUT: track 167.7 -> 0.00 mm
- net N$1: track 152.5 -> 0.00 mm
- net MOO: track 143.7 -> 0.00 mm
- net MAC: track 111.2 -> 0.00 mm
- net MA: track 101.4 -> 0.00 mm
- net N$2: track 89.7 -> 0.00 mm
- net MKK: track 86.2 -> 0.00 mm, vias 1 -> 0
- net N$3: track 38.4 -> 0.00 mm
- net MAD: track 38.3 -> 0.00 mm
- net MBB: track 35.9 -> 0.00 mm
- net ML: track 35.5 -> 0.00 mm
- net 18V: track 26.8 -> 0.00 mm
- net N$6: track 11.0 -> 0.00 mm
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- removed copper zone on layer 1, net GND
- removed copper zone on layer 16, net GND
Other:
- board size 140 x 80 mm -> 100 x 100 mm

Commit message: power
Parts:
- removed JETSON1: 1N5908, diode:C4111-15
- removed R7: (no value), resistor-power:AC01
- moved U$1 109.2 mm to (2.00, 88.0)
Connections:
- removed net MA1: JETSON1.C, R7.2, U$1.SOURCE
- removed net N$5: JETSON18V-OUT1.P$1, U$1.DRAIN
- new net N$43: JET.L, R4.1, U$1.GATE, U$4.GATE
- net 18V: no longer JETSON1.A
- net MA: now also U$1.SOURCE
- net MAC: now also JETSON18V-OUT1.P$1; no longer U$4.DRAIN
- net N$4: now also U$1.DRAIN, U$4.DRAIN; no longer JET.L, R4.1, R7.1, U$1.GATE, U$4.GATE
